Commit message: The car model gets its real sensors: three cameras, the radar on the grill, the roof lidar
Ben (15 Oct): two cameras on top looking forward, one at the back looking
back, the mmWave radar on the grill, the lidar on top. The front right and
rear cameras are simulated and bridged as /sensors/camera/front_right and
/sensors/camera/rear; lidar_link and camera_rear_link are always in the
URDF, as the car has both. Positions are Ben's placement until Friday's tape
measure. The front cameras sit on the roof's front edge: inside Gazebo's
solid box they saw its walls.

The old repos had no mounting positions; the 2025-26 obstacle code read
/velodyne_points, so the lidar is probably a Velodyne.

sim-check now checks the two new cameras deliver pictures, and its lane run
no longer fails on Nav2's /map, which that run leaves out on purpose.

File: src/aav_description/urdf/aav.sensors.gazebo.xacro (robot description, xacro)
@@ -1,5 +1,5 @@
 <?xml version="1.0"?>
 <!--
-  The Gazebo car's camera and radar stand-in, and Gazebo's truth: included when sim:=true.
+  The Gazebo car's three cameras and radar stand-in, and Gazebo's truth: included when sim:=true.
   Each sensor sits at the URDF's own frame (vehicle.yaml), and its messages carry that
   frame, as the real devices' do. Only a world with the Sensors system renders them (the
@@ -8,4 +8,6 @@
     /aav/camera/image         gz.msgs.Image          -> /sensors/camera/front_left/image_raw
     /aav/camera/camera_info   gz.msgs.CameraInfo     -> /sensors/camera/front_left/camera_info
+    /aav/camera_right/...     the same               -> /sensors/camera/front_right/...
+    /aav/camera_rear/...      the same               -> /sensors/camera/rear/...
     /aav/radar/points         gz.msgs.PointCloudPacked -> /sensors/radar/points (best effort)
     /model/aav/truth          gz.msgs.Odometry       -> /vehicle/gazebo/truth
@@ -22,22 +24,29 @@
   <xacro:property name="camera_height" value="360"/>
   <xacro:property name="camera_focal" value="343.0"/>
-  <gazebo reference="camera_left_link">
-    <sensor name="camera_left" type="camera">
-      <always_on>1</always_on>
-      <update_rate>10</update_rate>
-      <topic>/aav/camera/image</topic>
-      <gz_frame_id>camera_left_link</gz_frame_id>
-      <camera>
-        <camera_info_topic>/aav/camera/camera_info</camera_info_topic>
-        <horizontal_fov>${2 * atan(camera_width / 2.0 / camera_focal)}</horizontal_fov>
-        <image>
-          <width>${camera_width}</width>
-          <height>${camera_height}</height>
-          <format>R8G8B8</format>
-        </image>
-        <clip><near>0.1</near><far>150</far></clip>
-      </camera>
-    </sensor>
-  </gazebo>
+  <xacro:macro name="sim_camera" params="link name topic">
+    <gazebo reference="${link}">
+      <sensor name="${name}" type="camera">
+        <always_on>1</always_on>
+        <update_rate>10</update_rate>
+        <topic>${topic}/image</topic>
+        <gz_frame_id>${link}</gz_frame_id>
+        <camera>
+          <camera_info_topic>${topic}/camera_info</camera_info_topic>
+          <horizontal_fov>${2 * atan(camera_width / 2.0 / camera_focal)}</horizontal_fov>
+          <image>
+            <width>${camera_width}</width>
+            <height>${camera_height}</height>
+            <format>R8G8B8</format>
+          </image>
+          <clip><near>0.1</near><far>150</far></clip>
+        </camera>
+      </sensor>
+    </gazebo>
+  </xacro:macro>
+  <!-- The car's three: two up top looking forward, one at the back looking back. All the
+       same lens, as the front ones are the same model; the rear one's is unknown (N4). -->
+  <xacro:sim_camera link="camera_left_link" name="camera_left" topic="/aav/camera"/>
+  <xacro:sim_camera link="camera_right_link" name="camera_right" topic="/aav/camera_right"/>
+  <xacro:sim_camera link="camera_rear_link" name="camera_rear" topic="/aav/camera_rear"/>
   <!-- A radar stand-in: a lidar shaped like the TI IWR6843AOP with ti_ros2_driver's
        cfg/base.cfg, as the bench's mock_radar is: 8.4 m, 120 degrees wide, a ray every
@@ -87,5 +96,4 @@
        Rays that hit nothing come back as inf, which Nav2 and PCL drop. -->
   <xacro:if value="$(arg lidar)">
-    <xacro:sensor_frame name="lidar_link"/>
     <gazebo reference="lidar_link">
       <sensor name="lidar" type="gpu_lidar">

File: src/aav_description/urdf/aav.urdf.xacro (robot description, xacro)
@@ -15,6 +15,6 @@
   <xacro:arg name="vehicle_config" default="$(find aav_description)/config/vehicle.yaml"/>
   <xacro:arg name="sim" default="false"/>
-  <!-- With sim: a simulated roof lidar on lidar_link (aav.sensors.gazebo.xacro). The car
-       has none, so it never appears without sim. -->
+  <!-- With sim: the roof lidar is simulated too (aav.sensors.gazebo.xacro). Its frame,
+       lidar_link, is always there: the car has one. -->
   <xacro:arg name="lidar" default="false"/>
   <xacro:property name="cfg" value="${xacro.load_yaml('$(arg vehicle_config)')}"/>
@@ -182,4 +182,6 @@
   <xacro:sensor_frame name="camera_left_link"/>
   <xacro:sensor_frame name="camera_right_link"/>
+  <xacro:sensor_frame name="camera_rear_link"/>
+  <xacro:sensor_frame name="lidar_link"/>
   <xacro:if value="$(arg sim)">
     <xacro:include filename="$(find aav_description)/urdf/aav.gazebo.xacro"/>
