Commit message: Gazebo steers as vehicle.yaml says: 0.022 s behind the model, was 0.111 (TODO 52c)
Gazebo's own steering added a 0.11 s lag after the actuator model, more than
vehicle.yaml's steer_lag itself, so the simulator steered later than the car the
model describes. Raising steer_p_gain alone made it worse: the URDF's steering
joints had a 1.0 rad/s speed limit, which Gazebo enforces, and its wheels then
turned at only 0.63 rad/s, slower than the model's 0.8. So the joints' limit goes
to 5.0 rad/s (the model limits, not Gazebo) and steer_p_gain 10 -> 100. Measured
in Gazebo with actuator-test steer-rate --sim and the new tools/gazebo_steering.py
(the joints against the model's angle, fitted by analysis.fit_follower).

Gain 100 rather than taking 0.1 s off the adapter's lag (11 ms nearer): the
adapter's /vehicle/steering stays the wheels' angle, and a measured steer_lag
needs no change in the xacro. A test keeps Gazebo's extra lag under a quarter of
steer_lag and the joints' speed limit over 4 x steer_rate.

File: ros/bringup/aav_description/urdf/aav.gazebo.xacro (robot description, xacro)
@@ -27,5 +27,5 @@
            gazebo_steering_limit). Missing: xacro stops here rather than steer short. -->
       <steering_limit>${float('$(arg gz_steering_limit)')}</steering_limit>
-      <steer_p_gain>10.0</steer_p_gain>  <!-- the default lags over 1 s, and Nav2 weaves -->
+      <steer_p_gain>100.0</steer_p_gain>
       <wheel_base>${L}</wheel_base>
       <wheel_separation>${T}</wheel_separation>

File: ros/bringup/aav_description/urdf/aav.urdf.xacro (robot description, xacro)
@@ -154,6 +154,8 @@
       <origin xyz="${L} ${y} ${R}"/>
       <axis xyz="0 0 1"/>
-      <!-- The inner wheel turns further than the virtual centre wheel. -->
-      <limit lower="${-1.3 * max_steer}" upper="${1.3 * max_steer}" effort="100" velocity="1.0"/>
+      <!-- The inner wheel turns further than the virtual centre wheel. velocity: Gazebo
+           holds the joint to it, and at 1.0 its wheels turned only 0.63 rad/s, slower than
+           the actuator model's steer_rate (TODO 52c): far over it, so the model limits. -->
+      <limit lower="${-1.3 * max_steer}" upper="${1.3 * max_steer}" effort="100" velocity="5.0"/>
     </joint>
     <xacro:wheel name="${name}" side="${side}"/>
